File: PCB/JSDM Wemos Mini DS3231 HUB12 & 08 Single/JSDM Wemos DS3231 Single Layer.sch (EAGLE design)
At the start: 14 parts, among them X1 PSU

Commit message: Update Skematik ESP8266
Parts:
- R2: value 1K -> 2K2
Connections:
- net TOMBOL renamed WIPING
