File: PCB/JSDM ESP32 DevKit DS3231 HUB12 & 08 Single/JSDM ESP32 DevKit DS3231 HUB12 & 08 Single.sch (EAGLE design)
At the start: 14 parts, among them X1 PSU

Commit message: JSDM PCB Single Layer ESP8266 + ESP32
Desain PCB SIngle Layer versi:
- Wemos D1 mini HUB12 + HUB08
- Wemos D1 Mini 3x HUB12
- ESP32 Devkit HUB12 + HUB08
- ESP32 Devkit Mini 3x HUB12
Parts:
- removed R1: 10K, FansElectronics-RCL:R-EU_0207/12
- removed R3: PROG, FansElectronics-RCL:R-EU_M0805
- removed WEMOS1: (no value), esp8266modules:WEMOS-D1-MINI
- added ESP1: ESP32_DEVKIT, DOIT_ESP32_DEVKIT:ESP32_DEVKIT
- added S1: WIPE, FansElectronics-Switch:TACT-6X6OCT
- C1: value (none) -> 10uF
- JP3: value (none) -> MUROTTAL; device FansElectronics-Header:PINHD-1X2 -> FansElectronics-Header:PINHD-1X6
- R2: value 2K2 -> 1K; device FansElectronics-RCL:R-EU_0207/7 -> FansElectronics-RCL:R-EU_0207/10
Connections:
- removed net D0: IC1.A2, WEMOS1.D0
- removed net D3: IC1.A7, WEMOS1.D3
- removed net D4: IC1.A4, WEMOS1.D4
- removed net D5: IC1.A6, WEMOS1.D5
- removed net D6: IC1.A3, WEMOS1.D6
- removed net D7: IC1.A8, WEMOS1.D7
- removed net D8: IC1.A1, WEMOS1.D8
- removed net N$1: R1.2, WEMOS1.3V3
- removed net N$6: R2.2, R3.2
- removed net RX: IC1.A5, WEMOS1.RX
- removed net TX: R3.1, WEMOS1.TX
- removed net WIPING: JP3.2, R1.1, WEMOS1.A0
- new net +3V3: ESP1.3V3
- new net BUZZER: ESP1.D15, R2.2
- new net DMD_A: ESP1.RX2, IC1.A2
- new net DMD_B: ESP1.D14, IC1.A3
- new net DMD_C: ESP1.TX2, IC1.A4
- new net DMD_CLK: ESP1.D18, IC1.A6
- new net DMD_D: ESP1.D5, IC1.A5
- new net DMD_NOE: ESP1.D4, IC1.A1
- new net DMD_R1: ESP1.D23, IC1.A8
- new net DMD_STB: ESP1.D19, IC1.A7
- new net MP3_RX: ESP1.D25, JP3.2
- new net MP3_TX: ESP1.D33, JP3.1
- new net RELAY1: ESP1.D27, JP3.4
- new net RELAY2: ESP1.D26, JP3.3
- new net WIPE: ESP1.D13, S1.S
- net +5V: now also ESP1.VIN, JP3.5; no longer WEMOS1.5V
- net GND: now also ESP1.GND@1, ESP1.GND@2, JP3.6, S1.P, S1.P1; no longer JP3.1, WEMOS1.GND
- net SCL: now also ESP1.D22; no longer WEMOS1.D1
- net SDA: now also ESP1.D21; no longer WEMOS1.D2
Other:
- note added: "Irfan Indra Kurniawan @Vean"
- note added: "JSDM ESP32 DevKit DS3231 HUB12 & 08 Single - V1.0"
- note removed: "Controller Jadwal Sholat WEMOS D1 ESP8266 - V1"
- note removed: "Irfan Indra Kurniawan"
- moved on the sheet: C1, IC1, JP1, JP2, JP4, MOD2, R2, SG1, T1, X1
